Commit message: robot able to move

File: robot.urdf.xacro (robot description, xacro)
@@ -60,4 +60,24 @@
       <origin xyz="${baselen*reflect/3} 0 -${wheeldiam/2+.05}" rpy="0 0 0"/>
     </joint>
+    <!-- This block provides the simulator (Gazebo) with information on a few additional
+    physical properties. See http://gazebosim.org/tutorials/?tut=ros_urdf for more-->
+    <gazebo reference="${prefix}_${suffix}_wheel">
+      <mu1 value="400.0"/>
+      <mu2 value="300.0"/>
+      <kp value="100000000.0" />
+      <kd value="1.0" />
+      <material>Gazebo/Grey</material>
+    </gazebo>
+    <!-- This block connects the wheel joint to an actuator (motor), which informs both
+    simulation and visualization of the robot -->
+    <transmission name="${prefix}_${suffix}_wheel_trans">
+      <type>transmission_interface/SimpleTransmission</type>
+      <actuator name="${prefix}_${suffix}_wheel_motor">
+        <mechanicalReduction>1</mechanicalReduction>
+      </actuator>
+      <joint name="${prefix}_${suffix}_wheel_joint">
+        <hardwareInterface>VelocityJointInterface</hardwareInterface>
+      </joint>
+    </transmission>
   </xacro:macro>
   <xacro:macro name="leg" params="prefix reflect">

Commit message: custom bot can move faster now

File: robot.urdf.xacro (robot description, xacro)
@@ -6,5 +6,5 @@
   <xacro:property name="bodylen" value="0.6" />
   <xacro:property name="baselen" value="0.4" />
-  <xacro:property name="wheeldiam" value="0.07" />
+  <xacro:property name="wheeldiam" value="0.1" />
   <xacro:property name="pi" value="3.1415" />
   <material name="blue">

Commit message: bot changed to a car type

File: robot.urdf.xacro (robot description, xacro)
@@ -1,8 +1,8 @@
 <?xml version="1.0"?>
-<robot name="macroed" xmlns:xacro="http://ros.org/wiki/xacro">
-  <xacro:property name="width" value="0.2" />
-  <xacro:property name="leglen" value="0.6" />
-  <xacro:property name="polelen" value="0.2" />
-  <xacro:property name="bodylen" value="0.6" />
+<robot name="car" xmlns:xacro="http://ros.org/wiki/xacro">
+  <xacro:property name="width" value="0.1" />
+  <xacro:property name="leglen" value="0.1" />
+  <xacro:property name="polelen" value="0.0" />
+  <xacro:property name="bodylen" value="0.2" />
   <xacro:property name="baselen" value="0.4" />
   <xacro:property name="wheeldiam" value="0.1" />
@@ -26,12 +26,14 @@
     <visual>
       <geometry>
-        <cylinder radius="${width}" length="${bodylen}"/>
+        <box size="${baselen} ${bodylen} 0.1"/>
       </geometry>
+      <origin xyz="0 0 0.15"/>
       <material name="blue"/>
     </visual>
     <collision>
       <geometry>
-        <cylinder radius="${width}" length="${bodylen}"/>
+        <box size="${baselen} ${bodylen} 0.1"/>
       </geometry>
+      <origin xyz="0 0 0.15" />
     </collision>
     <xacro:default_inertial mass="10"/>
@@ -67,5 +69,5 @@
       <kp value="100000000.0" />
       <kd value="1.0" />
-      <material>Gazebo/Grey</material>
+      <material>Gazebo/Orange</material>
     </gazebo>
     <!-- This block connects the wheel joint to an actuator (motor), which informs both
@@ -85,5 +87,5 @@
       <visual>
         <geometry>
-          <box size="${leglen} 0.1 0.2"/>
+          <box size="${leglen} 0.0 0.0"/>
         </geometry>
         <origin xyz="0 0 -${leglen/2}" rpy="0 ${pi/2} 0"/>
@@ -92,5 +94,5 @@
       <collision>
         <geometry>
-          <box size="${leglen} 0.1 0.2"/>
+          <box size="${leglen} 0.0 0.0"/>
         </geometry>
         <origin xyz="0 0 -${leglen/2}" rpy="0 ${pi/2} 0"/>
@@ -127,54 +129,4 @@
   <xacro:leg prefix="right" reflect="-1" />
   <xacro:leg prefix="left" reflect="1" />
-  <link name="head">
-    <visual>
-      <geometry>
-        <sphere radius="${width}"/>
-      </geometry>
-      <material name="white"/>
-    </visual>
-    <collision>
-      <geometry>
-        <sphere radius="${width}"/>
-      </geometry>
-    </collision>
-    <xacro:default_inertial mass="2"/>
-  </link>
-  <joint name="head_swivel" type="continuous">
-    <parent link="base_link"/>
-    <child link="head"/>
-    <axis xyz="0 0 1"/>
-    <origin xyz="0 0 ${bodylen/2}"/>
-    <limit effort="30" velocity="1.0"/>
-  </joint>
-  <transmission name="head_swivel_trans">
-    <type>transmission_interface/SimpleTransmission</type>
-    <actuator name="$head_swivel_motor">
-      <mechanicalReduction>1</mechanicalReduction>
-    </actuator>
-    <joint name="head_swivel">
-      <hardwareInterface>hardware_interface/PositionJointInterface</hardwareInterface>
-    </joint>
-  </transmission>
-  <link name="box">
-    <visual>
-      <geometry>
-        <box size="0.08 0.08 0.08"/>
-      </geometry>
-      <material name="blue"/>
-      <origin xyz="-0.04 0 0"/>
-    </visual>
-    <collision>
-      <geometry>
-        <box size="0.08 0.08 0.08"/>
-      </geometry>
-    </collision>
-    <xacro:default_inertial mass="1"/>
-  </link>
-  <joint name="tobox" type="fixed">
-    <parent link="head"/>
-    <child link="box"/>
-    <origin xyz="${.707*width+0.04} 0 ${.707*width}"/>
-  </joint>
   <!-- Gazebo plugin for ROS Control -->
   <gazebo>

Commit message: changed colour for better visualization

File: robot.urdf.xacro (robot description, xacro)
@@ -29,5 +29,5 @@
       </geometry>
       <origin xyz="0 0 0.15"/>
-      <material name="blue"/>
+      <material name="black"/>
     </visual>
     <collision>
@@ -39,4 +39,7 @@
     <xacro:default_inertial mass="10"/>
   </link>
+  <gazebo reference="base_link">
+    <material>Gazebo/Black</material>
+  </gazebo>
   <xacro:macro name="wheel" params="prefix suffix reflect">
     <link name="${prefix}_${suffix}_wheel">
@@ -90,5 +93,5 @@
         </geometry>
         <origin xyz="0 0 -${leglen/2}" rpy="0 ${pi/2} 0"/>
-        <material name="white"/>
+        <material name="blue"/>
       </visual>
       <collision>
@@ -110,5 +113,5 @@
           <box size="${baselen} 0.1 0.1"/>
         </geometry>
-        <material name="white"/>
+        <material name="blue"/>
       </visual>
       <collision>
@@ -126,4 +129,10 @@
     <xacro:wheel prefix="${prefix}" suffix="front" reflect="1"/>
     <xacro:wheel prefix="${prefix}" suffix="back" reflect="-1"/>
+    <gazebo reference="${prefix}_leg">
+      <material>Gazebo/Blue</material>
+    </gazebo>
+    <gazebo reference="${prefix}_base">
+      <material>Gazebo/Blue</material>
+    </gazebo>
   </xacro:macro>
   <xacro:leg prefix="right" reflect="-1" />

Commit message: resolved odom initialization issue

File: robot.urdf.xacro (robot description, xacro)
@@ -1,4 +1,5 @@
 <?xml version="1.0"?>
 <robot name="car" xmlns:xacro="http://ros.org/wiki/xacro">
+  <xacro:arg name="robot_name" default="car"/>
   <xacro:property name="width" value="0.1" />
   <xacro:property name="leglen" value="0.1" />
@@ -138,13 +139,29 @@
   <xacro:leg prefix="right" reflect="-1" />
   <xacro:leg prefix="left" reflect="1" />
+  <!-- <dummy link> -->
+  <link name="map" />
+  <link name="odom" />
+  <joint name="map_joint" type="fixed">
+    <parent link="map" />
+    <child link="odom" />
+    <origin xyz="0.0 0.0 0.0" rpy="0.0 0.0 0.0" />
+  </joint>
+  <link name="odom" />
+  <joint name="odom_joint" type="fixed">
+    <parent link="odom" />
+    <child link="base_link" />
+    <origin xyz="0.0 0.0 0.0" rpy="0.0 0.0 0.0" />
+  </joint>
   <!-- Gazebo plugin for ROS Control -->
   <gazebo>
     <plugin name="gazebo_ros_control" filename="libgazebo_ros_control.so">
-    <!-- output -->
-    <publish_odom>true</publish_odom>
-    <publish_odom_tf>false</publish_odom_tf>
-    <publish_wheel_tf>true</publish_wheel_tf>
-    <odometry_frame>/odom</odometry_frame>
-    <robot_base_frame>/base_link</robot_base_frame>
+    </plugin>
+    <plugin name="object_controller" filename="libgazebo_ros_planar_move.so">
+      <commandTopic>cmd_vel</commandTopic>
+      <odometryTopic>odom</odometryTopic>
+      <odometryFrame>odom</odometryFrame>
+      <odometryRate>50.0</odometryRate>
+      <robotBaseFrame>base_link</robotBaseFrame>
+      <cmdTimeout>1.0</cmdTimeout>
     </plugin>
   </gazebo>

Commit message: stresssss

File: robot.urdf.xacro (robot description, xacro)
@@ -1,5 +1,4 @@
 <?xml version="1.0"?>
 <robot name="car" xmlns:xacro="http://ros.org/wiki/xacro">
-  <xacro:arg name="robot_name" default="car"/>
   <xacro:property name="width" value="0.1" />
   <xacro:property name="leglen" value="0.1" />
@@ -139,5 +138,5 @@
   <xacro:leg prefix="right" reflect="-1" />
   <xacro:leg prefix="left" reflect="1" />
-  <!-- <dummy link> -->
+  <!-- <dummy links>
   <link name="map" />
   <link name="odom" />
@@ -146,15 +145,17 @@
     <child link="odom" />
     <origin xyz="0.0 0.0 0.0" rpy="0.0 0.0 0.0" />
-  </joint>
-  <link name="odom" />
-  <joint name="odom_joint" type="fixed">
+  </joint> -->
+  <!-- <link name="base_link"/> -->
+  <!-- <joint name="odom_joint" type="fixed">
     <parent link="odom" />
     <child link="base_link" />
     <origin xyz="0.0 0.0 0.0" rpy="0.0 0.0 0.0" />
-  </joint>
+  </joint> -->
   <!-- Gazebo plugin for ROS Control -->
   <gazebo>
     <plugin name="gazebo_ros_control" filename="libgazebo_ros_control.so">
     </plugin>
+  </gazebo>
+  <!-- <gazebo>
     <plugin name="object_controller" filename="libgazebo_ros_planar_move.so">
       <commandTopic>cmd_vel</commandTopic>
@@ -165,4 +166,4 @@
       <cmdTimeout>1.0</cmdTimeout>
     </plugin>
-  </gazebo>
+  </gazebo> -->
 </robot>

Commit message: basic setup restored

File: robot.urdf.xacro (robot description, xacro)
@@ -6,5 +6,5 @@
   <xacro:property name="bodylen" value="0.2" />
   <xacro:property name="baselen" value="0.4" />
-  <xacro:property name="wheeldiam" value="0.1" />
+  <xacro:property name="wheeldiam" value="0.14" />
   <xacro:property name="pi" value="3.1415" />
   <material name="blue">
@@ -120,5 +120,5 @@
         </geometry>
       </collision>
-      <xacro:default_inertial mass="10"/>
+      <xacro:default_inertial mass="20"/>
     </link>
     <joint name="${prefix}_base_joint" type="fixed">

Commit message: shifted to two-wheel with castor wheel bot

File: robot.urdf.xacro (robot description, xacro)
@@ -1,11 +1,14 @@
 <?xml version="1.0"?>
-<robot name="car" xmlns:xacro="http://ros.org/wiki/xacro">
-  <xacro:property name="width" value="0.1" />
-  <xacro:property name="leglen" value="0.1" />
-  <xacro:property name="polelen" value="0.0" />
-  <xacro:property name="bodylen" value="0.2" />
-  <xacro:property name="baselen" value="0.4" />
-  <xacro:property name="wheeldiam" value="0.14" />
-  <xacro:property name="pi" value="3.1415" />
+<robot xmlns:xacro="http://www.ros.org/wiki/xacro" name="ros">
+  <xacro:property name="base_width" value="0.16"/>
+  <xacro:property name="base_len" value="0.16"/>
+  <xacro:property name="wheel_radius" value="0.05"/>
+  <xacro:property name="base_wheel_gap" value="0.007"/>
+  <xacro:property name="wheel_separation" value="0.15"/>
+  <xacro:property name="wheel_joint_offset" value="0.02"/>
+  <xacro:property name="caster_wheel_radius" value="${wheel_radius/2}"/>
+  <xacro:property name="caster_wheel_mass" value="0.001"/>
+  <xacro:property name="caster_wheel_joint_offset" value="-0.052"/>
+  <!--Color Properties-->
   <material name="blue">
     <color rgba="0 0 0.8 1"/>
@@ -17,153 +20,140 @@
     <color rgba="1 1 1 1"/>
   </material>
-  <xacro:macro name="default_inertial" params="mass">
+  <material name="red">
+    <color rgba="0.8 0.0 0.0 1.0"/>
+  </material>
+  <!--Interial macros-->
+  <xacro:macro name="cylinder_inertia" params="m r h">
     <inertial>
-      <mass value="${mass}" />
-      <inertia ixx="1.0" ixy="0.0" ixz="0.0" iyy="1.0" iyz="0.0" izz="1.0" />
+      <mass value="${m}"/>
+      <inertia ixx="${m*(3*r*r+h*h)/12}" ixy = "0" ixz = "0" iyy="${m*(3*r*r+h*h)/12}" iyz = "0" izz="${m*r*r/2}"/>
     </inertial>
   </xacro:macro>
+  <xacro:macro name="box_inertia" params="m w h d">
+    <inertial>
+      <mass value="${m}"/>
+      <inertia ixx="${m / 12.0 * (d*d + h*h)}" ixy="0.0" ixz="0.0" iyy="${m / 12.0 * (w*w + h*h)}" iyz="0.0" izz="${m / 12.0 * (w*w + d*d)}"/>
+    </inertial>
+  </xacro:macro>
+  <xacro:macro name="sphere_inertia" params="m r">
+    <inertial>
+      <mass value="${m}"/>
+      <inertia ixx="${2.0*m*(r*r)/5.0}" ixy="0.0" ixz="0.0" iyy="${2.0*m*(r*r)/5.0}" iyz="0.0" izz="${2.0*m*(r*r)/5.0}"/>
+    </inertial>
+  </xacro:macro>
+  <!--Base Footprint-->
+  <link name="base_footprint">
+    <xacro:box_inertia m="10" w="0.001" h="0.001" d="0.001"/>
+    <visual>
+        <origin xyz="0 0 0" rpy="0 0 0" />
+        <geometry>
+            <box size="0.001 0.001 0.001" />
+        </geometry>
+    </visual>
+  </link>
+  <!--Base link-->
   <link name="base_link">
+    <xacro:box_inertia m="10" w="${base_len}" h="${base_width}" d="0.05"/>
     <visual>
       <geometry>
-        <box size="${baselen} ${bodylen} 0.1"/>
+        <box size="${base_len} ${base_width} 0.05"/>
       </geometry>
-      <origin xyz="0 0 0.15"/>
       <material name="black"/>
     </visual>
     <collision>
       <geometry>
-        <box size="${baselen} ${bodylen} 0.1"/>
+        <box size="${base_len} ${base_width} 0.05"/>
       </geometry>
-      <origin xyz="0 0 0.15" />
     </collision>
-    <xacro:default_inertial mass="10"/>
   </link>
   <gazebo reference="base_link">
-    <material>Gazebo/Black</material>
+    <material>Gazebo/Blue</material>
   </gazebo>
-  <xacro:macro name="wheel" params="prefix suffix reflect">
-    <link name="${prefix}_${suffix}_wheel">
+  <!--base_link to base_footprint Joint-->
+  <joint name="base_link_joint" type="fixed">
+    <origin xyz="0 0 ${wheel_radius + 0.005}" rpy="0 0 0" />
+    <parent link="base_footprint"/>
+    <child link="base_link" />
+  </joint>
+  <!--Wheel link & joint macro-->
+  <xacro:macro name="wheel" params="prefix reflect">
+    <link name="${prefix}_wheel">
       <visual>
-        <origin xyz="0 0 0" rpy="${pi/2} 0 0" />
+        <origin xyz="0 0 0" rpy="${pi/2} 0 0"/>
         <geometry>
-          <cylinder radius="${wheeldiam/2}" length="0.1"/>
+          <cylinder radius="${wheel_radius}" length="0.005"/>
         </geometry>
-        <material name="black"/>
+        <material name="red"/>
       </visual>
       <collision>
-        <origin xyz="0 0 0" rpy="${pi/2} 0 0" />
+        <origin xyz="0 0 0" rpy="${pi/2} 0 0"/>
         <geometry>
-          <cylinder radius="${wheeldiam/2}" length="0.1"/>
+          <cylinder radius="${wheel_radius}" length="0.005"/>
         </geometry>
       </collision>
-      <xacro:default_inertial mass="1"/>
+      <xacro:cylinder_inertia m="10" r="${wheel_radius}" h="0.005"/>
     </link>
-    <joint name="${prefix}_${suffix}_wheel_joint" type="continuous">
+    <joint name="${prefix}_wheel_joint" type="continuous">
       <axis xyz="0 1 0" rpy="0 0 0" />
-      <parent link="${prefix}_base"/>
-      <child link="${prefix}_${suffix}_wheel"/>
-      <origin xyz="${baselen*reflect/3} 0 -${wheeldiam/2+.05}" rpy="0 0 0"/>
+      <parent link="base_link"/>
+      <child link="${prefix}_wheel"/>
+      <origin xyz="${wheel_joint_offset} ${((base_width/2)+base_wheel_gap)*reflect} -0.005" rpy="0 0 0"/>
     </joint>
-    <!-- This block provides the simulator (Gazebo) with information on a few additional
-    physical properties. See http://gazebosim.org/tutorials/?tut=ros_urdf for more-->
-    <gazebo reference="${prefix}_${suffix}_wheel">
-      <mu1 value="400.0"/>
-      <mu2 value="300.0"/>
-      <kp value="100000000.0" />
+    <gazebo reference="${prefix}_wheel">
+      <kp value="1000000.0" />
       <kd value="1.0" />
       <material>Gazebo/Orange</material>
     </gazebo>
-    <!-- This block connects the wheel joint to an actuator (motor), which informs both
-    simulation and visualization of the robot -->
-    <transmission name="${prefix}_${suffix}_wheel_trans">
-      <type>transmission_interface/SimpleTransmission</type>
-      <actuator name="${prefix}_${suffix}_wheel_motor">
-        <mechanicalReduction>1</mechanicalReduction>
-      </actuator>
-      <joint name="${prefix}_${suffix}_wheel_joint">
-        <hardwareInterface>hardware_interface/VelocityJointInterface</hardwareInterface>
-      </joint>
-    </transmission>
   </xacro:macro>
-  <xacro:macro name="leg" params="prefix reflect">
-    <link name="${prefix}_leg">
-      <visual>
-        <geometry>
-          <box size="${leglen} 0.0 0.0"/>
-        </geometry>
-        <origin xyz="0 0 -${leglen/2}" rpy="0 ${pi/2} 0"/>
-        <material name="blue"/>
-      </visual>
-      <collision>
-        <geometry>
-          <box size="${leglen} 0.0 0.0"/>
-        </geometry>
-        <origin xyz="0 0 -${leglen/2}" rpy="0 ${pi/2} 0"/>
-      </collision>
-      <xacro:default_inertial mass="10"/>
-    </link>
-    <joint name="base_to_${prefix}_leg" type="fixed">
-      <parent link="base_link"/>
-      <child link="${prefix}_leg"/>
-      <origin xyz="0 ${reflect*(width+.02)} 0.25" />
-    </joint>
-    <link name="${prefix}_base">
-      <visual>
-        <geometry>
-          <box size="${baselen} 0.1 0.1"/>
-        </geometry>
-        <material name="blue"/>
-      </visual>
-      <collision>
-        <geometry>
-          <box size="${baselen} 0.1 0.1"/>
-        </geometry>
-      </collision>
-      <xacro:default_inertial mass="20"/>
-    </link>
-    <joint name="${prefix}_base_joint" type="fixed">
-      <parent link="${prefix}_leg"/>
-      <child link="${prefix}_base"/>
-      <origin xyz="0 0 ${-leglen}" />
-    </joint>
-    <xacro:wheel prefix="${prefix}" suffix="front" reflect="1"/>
-    <xacro:wheel prefix="${prefix}" suffix="back" reflect="-1"/>
-    <gazebo reference="${prefix}_leg">
-      <material>Gazebo/Blue</material>
-    </gazebo>
-    <gazebo reference="${prefix}_base">
-      <material>Gazebo/Blue</material>
-    </gazebo>
-  </xacro:macro>
-  <xacro:leg prefix="right" reflect="-1" />
-  <xacro:leg prefix="left" reflect="1" />
-  <!-- <dummy links>
-  <link name="map" />
-  <link name="odom" />
-  <joint name="map_joint" type="fixed">
-    <parent link="map" />
-    <child link="odom" />
-    <origin xyz="0.0 0.0 0.0" rpy="0.0 0.0 0.0" />
-  </joint> -->
-  <!-- <link name="base_link"/> -->
-  <!-- <joint name="odom_joint" type="fixed">
-    <parent link="odom" />
-    <child link="base_link" />
-    <origin xyz="0.0 0.0 0.0" rpy="0.0 0.0 0.0" />
-  </joint> -->
-  <!-- Gazebo plugin for ROS Control -->
+  <!--Create Left & Right Wheel links/joints-->
+  <xacro:wheel prefix="left" reflect="1"/>
+  <xacro:wheel prefix="right" reflect="-1"/>
+  <!--Caster Wheel Link-->
+  <link name="caster_wheel">
+    <visual>
+      <origin xyz="0 0 0" rpy="0 0 0"/>
+      <geometry>
+        <sphere radius="${caster_wheel_radius}"/>
+      </geometry>
+      <material name="blue"/>
+    </visual>
+    <collision>
+      <origin xyz="0 0 0" rpy="0 0 0"/>
+      <geometry>
+        <sphere radius="${caster_wheel_radius}"/>
+      </geometry>
+    </collision>
+    <xacro:sphere_inertia m="10" r="${caster_wheel_radius}"/>
+  </link>
+  <!--Caster Wheel Joint-->
+  <joint name="caster_wheel_joint" type="continuous">
+    <axis xyz="0 1 0" rpy="0 0 0" />
+    <parent link="base_link"/>
+    <child link="caster_wheel"/>
+    <origin xyz="${caster_wheel_joint_offset} 0 -${caster_wheel_radius+0.005}" rpy="0 0 0"/>
+  </joint>
   <gazebo>
-    <plugin name="gazebo_ros_control" filename="libgazebo_ros_control.so">
+    <plugin name="differential_drive_controller" filename="libgazebo_ros_diff_drive.so">
+      <alwaysOn>false</alwaysOn>
+      <legacyMode>false</legacyMode>
+      <updateRate>20</updateRate>
+      <leftJoint>left_wheel_joint</leftJoint>
+      <rightJoint>right_wheel_joint</rightJoint>
+      <wheelSeparation>${wheel_separation}</wheelSeparation>
+      <wheelDiameter>${wheel_radius * 2}</wheelDiameter>
+      <torque>20</torque>
+      <commandTopic>/cmd_vel</commandTopic>
+      <odometryTopic>/odom</odometryTopic>
+      <odometryFrame>odom</odometryFrame>
+      <robotBaseFrame>base_footprint</robotBaseFrame>
+      <rosDebugLevel>Debug</rosDebugLevel>
+      <publishWheelTF>true</publishWheelTF>
+      <publishOdomTF>true</publishOdomTF>
+      <publishWheelJointState>true</publishWheelJointState>
+      <wheelAcceleration>5</wheelAcceleration>
+      <wheelTorque>20</wheelTorque>
+      <publishTf>1</publishTf>
+      <odometrySource>encoder</odometrySource>
     </plugin>
   </gazebo>
-  <!-- <gazebo>
-    <plugin name="object_controller" filename="libgazebo_ros_planar_move.so">
-      <commandTopic>cmd_vel</commandTopic>
-      <odometryTopic>odom</odometryTopic>
-      <odometryFrame>odom</odometryFrame>
-      <odometryRate>50.0</odometryRate>
-      <robotBaseFrame>base_link</robotBaseFrame>
-      <cmdTimeout>1.0</cmdTimeout>
-    </plugin>
-  </gazebo> -->
 </robot>
