Commit message: new robot ready

File: robot.urdf.xacro (robot description, xacro)
@@ -1,12 +1,12 @@
 <?xml version="1.0"?>
-<robot xmlns:xacro="http://www.ros.org/wiki/xacro" name="ros">
-  <xacro:property name="base_width" value="0.16"/>
-  <xacro:property name="base_len" value="0.16"/>
-  <xacro:property name="wheel_radius" value="0.05"/>
+<robot xmlns:xacro="http://www.ros.org/wiki/xacro" name="car">
+  <xacro:property name="base_width" value="0.33"/>
+  <xacro:property name="base_len" value="0.4"/>
+  <xacro:property name="wheel_radius" value="0.14"/>
   <xacro:property name="base_wheel_gap" value="0.007"/>
   <xacro:property name="wheel_separation" value="0.15"/>
   <xacro:property name="wheel_joint_offset" value="0.02"/>
   <xacro:property name="caster_wheel_radius" value="${wheel_radius/2}"/>
-  <xacro:property name="caster_wheel_mass" value="0.001"/>
+  <xacro:property name="caster_wheel_mass" value="0.01"/>
   <xacro:property name="caster_wheel_joint_offset" value="-0.052"/>
   <!--Color Properties-->
@@ -54,8 +54,8 @@
   <!--Base link-->
   <link name="base_link">
-    <xacro:box_inertia m="10" w="${base_len}" h="${base_width}" d="0.05"/>
+    <xacro:box_inertia m="10" w="${base_len}" h="${base_width}" d="0.1"/>
     <visual>
       <geometry>
-        <box size="${base_len} ${base_width} 0.05"/>
+        <box size="${base_len} ${base_width} 0.1"/>
       </geometry>
       <material name="black"/>
@@ -63,5 +63,5 @@
     <collision>
       <geometry>
-        <box size="${base_len} ${base_width} 0.05"/>
+        <box size="${base_len} ${base_width} 0.1"/>
       </geometry>
     </collision>
@@ -101,6 +101,4 @@
     </joint>
     <gazebo reference="${prefix}_wheel">
-      <kp value="1000000.0" />
-      <kd value="1.0" />
       <material>Gazebo/Orange</material>
     </gazebo>
@@ -143,7 +141,8 @@
       <wheelDiameter>${wheel_radius * 2}</wheelDiameter>
       <torque>20</torque>
-      <commandTopic>/cmd_vel</commandTopic>
-      <odometryTopic>/odom</odometryTopic>
+      <commandTopic>cmd_vel</commandTopic>
+      <odometryTopic>odom</odometryTopic>
       <odometryFrame>odom</odometryFrame>
+      <odometrySource>world</odometrySource>
       <robotBaseFrame>base_footprint</robotBaseFrame>
       <rosDebugLevel>Debug</rosDebugLevel>
@@ -154,5 +153,4 @@
       <wheelTorque>20</wheelTorque>
       <publishTf>1</publishTf>
-      <odometrySource>encoder</odometrySource>
     </plugin>
   </gazebo>
